Commit message: cleaned up comments a bit

File: Hector_ROS_Simulation/hector_description/xacro/const.xacro (robot description, xacro)
@@ -222,5 +222,5 @@
     <xacro:property name="twist_offset_y" value="0.0"/>
     <!--xacro:property name="twist_offset_z" value="-0.22"/-->
-    <xacro:property name="twist_offset_z" value="-0.045"/>
+    <xacro:property name="twist_offset_z" value="-0.062"/>
     <xacro:property name="twist_offset" value="0.019"/>
     <xacro:property name="twist_max" value="1.4"/>

File: Hector_ROS_Simulation/hector_description/xacro/leg.xacro (robot description, xacro)
@@ -18,5 +18,5 @@
         <link name="${name}_hip">
             <visual>
-                <origin rpy="0 0 0" xyz="0 0 0"/>
+                <origin rpy="0 0 0" xyz="0 0 0.02"/>
                 <xacro:if value="${(mirror_dae == True)}">
                     <geometry>

File: Hector_ROS_Simulation/hector_description/xacro/robot.xacro (robot description, xacro)
@@ -36,5 +36,5 @@
             <origin rpy="0 0 0" xyz="0 0 0"/>
             <geometry>
-                <mesh filename="package://hector_description/meshes/body.STL" scale="1 1 1"/>
+                <mesh filename="package://hector_description/meshes/body.stl" scale="1 1 1"/>
             </geometry>
             <material name="white"/>
@@ -113,5 +113,5 @@
         <parent link="trunk"/>
         <child link="head_link"/>
-        <origin rpy="0 ${PI} ${PI/2}" xyz="0.07 0.0458 0.315"/>
+        <origin rpy="0 ${PI} ${PI/2}" xyz="0.07 0.0458 0.3"/>
     </joint>
     <link name="head_link">
