Commit message: modified xacro for new arms

File: Hector_ROS_Simulation/hector_description/xacro/arm.xacro (robot description, xacro)
@@ -22,9 +22,22 @@
         </joint>
         <link name="${name}_twist">
-            <visual>
+            <!--
             <origin rpy="0 ${-PI/2.0} 0" xyz="0 0 0"/>
             <geometry>
                 <mesh filename="package://hector_description/meshes/hip_a1.dae" scale="1 1 1"/>
             </geometry>
+             -->
+            <visual>
+            <origin rpy="0 0 0" xyz="0 0 ${twist_offset_z}"/>
+            <xacro:if value="${(mirror_dae == True)}">
+            <geometry>
+                <mesh filename="package://hector_description/meshes/hector_arm/ShoulderYaw_L.stl" scale="1 1 1"/>
+            </geometry>
+            </xacro:if>
+            <xacro:if value="${(mirror_dae == False)}">
+            <geometry>
+                <mesh filename="package://hector_description/meshes/hector_arm/ShoulderYaw_R.stl" scale="1 1 1"/>
+            </geometry>
+            </xacro:if>
             <material name="orange"/>
             </visual>
@@ -49,4 +62,47 @@
             </inertial> -->
         </link>
+        <joint name="${name}_roll_joint" type="revolute">
+            <xacro:if value="${(mirror_dae == True)}">
+            <origin rpy="0 0 0" xyz="0.0 0.05 0.0"/>
+            </xacro:if>
+            <xacro:if value="${(mirror_dae == False)}">
+            <origin rpy="0 0 0" xyz="0.0 -0.05 0.0"/>
+            </xacro:if>
+            <parent link="${name}_twist"/>
+            <child link="${name}_roll"/>
+            <axis xyz="0 1 0"/>
+            <dynamics damping="${damping}" friction="${friction}"/>
+            <limit effort="${shoulder_torque_max}" velocity="${shoulder_velocity_max}" lower="${shoulder_min}" upper="${shoulder_max}"/>
+        </joint>
+        <link name="${name}_roll">
+            <visual>
+            <origin rpy="0 0 0" xyz="0 0 0"/>
+            <xacro:if value="${(mirror_dae == True)}">
+            <geometry>
+                <mesh filename="package://hector_description/meshes/hector_arm/ShoulderPitch_L.stl" scale="1 1 1"/>
+            </geometry>
+            </xacro:if>
+            <xacro:if value="${(mirror_dae == False)}">
+            <geometry>
+                <mesh filename="package://hector_description/meshes/hector_arm/ShoulderPitch_R.stl" scale="1 1 1"/>
+            </geometry>
+            </xacro:if>
+            <material name="orange"/>
+            </visual>
+           <collision>
+                <origin rpy="0 ${PI/2.0} 0" xyz="0 0 ${-shoulder_length/2.0}"/>
+                <geometry>
+                    <box size="${shoulder_length} ${shoulder_width} ${shoulder_height}"/>
+                </geometry>
+            </collision>
+            <inertial>
+                <origin rpy="0 0 0" xyz="${shoulder_com_x} ${shoulder_com_y*mirror} ${shoulder_com_z}"/>
+                <mass value="${shoulder_mass}"/>
+                <inertia
+                    ixx="${shoulder_ixx}" ixy="${shoulder_ixy*mirror}" ixz="${shoulder_ixz}"
+                    iyy="${shoulder_iyy}" iyz="${shoulder_iyz*mirror}"
+                    izz="${shoulder_izz}"/>
+            </inertial>
+        </link>
         <joint name="${name}_shoulder_joint" type="revolute">
             <xacro:if value="${(mirror_dae == True)}">
@@ -56,5 +112,5 @@
             <origin rpy="0 0 0" xyz="0.0 -0.0723 0.0"/>
             </xacro:if>
-            <parent link="${name}_twist"/>
+            <parent link="${name}_roll"/>
             <child link="${name}_shoulder"/>
             <axis xyz="0 1 0"/>
@@ -67,10 +123,12 @@
             <xacro:if value="${(mirror_dae == True)}">
             <geometry>
-                <mesh filename="package://hector_description/meshes/thigh_a1.dae" scale="1 1 1"/>
+                <!--mesh filename="package://hector_description/meshes/thigh_a1.dae" scale="1 1 1"/-->
+                <mesh filename="package://hector_description/meshes/hector_arm/UpperArmRoll_L.stl" scale="1 1 1"/>
             </geometry>
             </xacro:if>
             <xacro:if value="${(mirror_dae == False)}">
             <geometry>
-                <mesh filename="package://hector_description/meshes/thigh_mirror_a1.dae" scale="1 1 1"/>
+                <!--mesh filename="package://hector_description/meshes/thigh_mirror_a1.dae" scale="1 1 1"/-->
+                <mesh filename="package://hector_description/meshes/hector_arm/UpperArmRoll_R.stl" scale="1 1 1"/>
             </geometry>
             </xacro:if>
@@ -104,5 +162,6 @@
             <origin rpy="0 0 0" xyz="0 0 0"/>
             <geometry>
-                <mesh filename="package://hector_description/meshes/calf_a1.dae" scale="1 1 1"/>
+                <!--mesh filename="package://hector_description/meshes/calf_a1.dae" scale="1 1 1"/-->
+                <mesh filename="package://hector_description/meshes/hector_arm/ForeArmPitch.stl" scale="1 1 1"/>
             </geometry>
             <material name="orange"/>

File: Hector_ROS_Simulation/hector_description/xacro/arm_transmission.xacro (robot description, xacro)
@@ -9,4 +9,14 @@
             </joint>
             <actuator name="${name}_twist_motor">
+            <hardwareInterface>hardware_interface/EffortJointInterface</hardwareInterface>
+            <mechanicalReduction>1</mechanicalReduction>
+            </actuator>
+        </transmission>
+        <transmission name="${name}_roll_tran">
+            <type>transmission_interface/SimpleTransmission</type>
+            <joint name="${name}_roll_joint">
+            <hardwareInterface>hardware_interface/EffortJointInterface</hardwareInterface>
+            </joint>
+            <actuator name="${name}_roll_motor">
             <hardwareInterface>hardware_interface/EffortJointInterface</hardwareInterface>
             <mechanicalReduction>1</mechanicalReduction>

File: Hector_ROS_Simulation/hector_description/xacro/const.xacro (robot description, xacro)
@@ -221,5 +221,6 @@
     <xacro:property name="twist_offset_x" value="0.0"/>
     <xacro:property name="twist_offset_y" value="0.0"/>
-    <xacro:property name="twist_offset_z" value="-0.22"/>
+    <!--xacro:property name="twist_offset_z" value="-0.22"/-->
+    <xacro:property name="twist_offset_z" value="-0.05"/>
     <xacro:property name="twist_offset" value="0.019"/>
     <xacro:property name="twist_max" value="1.4"/>

Commit message: still changing arms

File: Hector_ROS_Simulation/hector_description/xacro/arm.xacro (robot description, xacro)
@@ -62,5 +62,5 @@
             </inertial> -->
         </link>
-        <joint name="${name}_roll_joint" type="revolute">
+        <joint name="${name}_shoulder_joint" type="revolute">
             <xacro:if value="${(mirror_dae == True)}">
             <origin rpy="0 0 0" xyz="0.0 0.05 0.0"/>
@@ -70,10 +70,10 @@
             </xacro:if>
             <parent link="${name}_twist"/>
-            <child link="${name}_roll"/>
+            <child link="${name}_shoulder"/>
             <axis xyz="0 1 0"/>
             <dynamics damping="${damping}" friction="${friction}"/>
             <limit effort="${shoulder_torque_max}" velocity="${shoulder_velocity_max}" lower="${shoulder_min}" upper="${shoulder_max}"/>
         </joint>
-        <link name="${name}_roll">
+        <link name="${name}_shoulder">
             <visual>
             <origin rpy="0 0 0" xyz="0 0 0"/>
@@ -105,23 +105,22 @@
             </inertial>
         </link>
-        <joint name="${name}_shoulder_joint" type="revolute">
+        <joint name="${name}_roll_joint" type="revolute">
             <xacro:if value="${(mirror_dae == True)}">
-            <origin rpy="0 0 0" xyz="0.0 0.0723 0.0"/>
+            <origin rpy="0 0 0" xyz="0.0 0.05 0.0"/>
             </xacro:if>
             <xacro:if value="${(mirror_dae == False)}">
-            <origin rpy="0 0 0" xyz="0.0 -0.0723 0.0"/>
+            <origin rpy="0 0 0" xyz="0.0 -0.05 0.0"/>
             </xacro:if>
-            <parent link="${name}_roll"/>
-            <child link="${name}_shoulder"/>
+            <parent link="${name}_shoulder"/>
+            <child link="${name}_roll"/>
             <axis xyz="0 1 0"/>
             <dynamics damping="${damping}" friction="${friction}"/>
             <limit effort="${shoulder_torque_max}" velocity="${shoulder_velocity_max}" lower="${shoulder_min}" upper="${shoulder_max}"/>
         </joint>
-        <link name="${name}_shoulder">
+        <link name="${name}_roll">
             <visual>
             <origin rpy="0 0 0" xyz="0 0 0"/>
             <xacro:if value="${(mirror_dae == True)}">
             <geometry>
-                <!--mesh filename="package://hector_description/meshes/thigh_a1.dae" scale="1 1 1"/-->
                 <mesh filename="package://hector_description/meshes/hector_arm/UpperArmRoll_L.stl" scale="1 1 1"/>
             </geometry>
@@ -129,5 +128,4 @@
             <xacro:if value="${(mirror_dae == False)}">
             <geometry>
-                <!--mesh filename="package://hector_description/meshes/thigh_mirror_a1.dae" scale="1 1 1"/-->
                 <mesh filename="package://hector_description/meshes/hector_arm/UpperArmRoll_R.stl" scale="1 1 1"/>
             </geometry>
@@ -152,5 +150,5 @@
         <joint name="${name}_elbow_joint" type="revolute">
             <origin rpy="0 -1.5 0" xyz="0.0 0.0 -0.205"/>
-            <parent link="${name}_shoulder"/>
+            <parent link="${name}_roll"/>
             <child link="${name}_elbow"/>
             <axis xyz="0 1 0"/>
@@ -162,5 +160,4 @@
             <origin rpy="0 0 0" xyz="0 0 0"/>
             <geometry>
-                <!--mesh filename="package://hector_description/meshes/calf_a1.dae" scale="1 1 1"/-->
                 <mesh filename="package://hector_description/meshes/hector_arm/ForeArmPitch.stl" scale="1 1 1"/>
             </geometry>

File: Hector_ROS_Simulation/hector_description/xacro/transmission.xacro (robot description, xacro)
@@ -75,4 +75,14 @@
             </actuator>
         </transmission>
+         <transmission name="${name}_roll_tran">
+            <type>transmission_interface/SimpleTransmission</type>
+            <joint name="${name}_roll_joint">
+            <hardwareInterface>hardware_interface/EffortJointInterface</hardwareInterface>
+            </joint>
+            <actuator name="${name}_roll_motor">
+            <hardwareInterface>hardware_interface/EffortJointInterface</hardwareInterface>
+            <mechanicalReduction>1</mechanicalReduction>
+            </actuator>
+        </transmission>
         <transmission name="${name}_elbow_tran">
             <type>transmission_interface/SimpleTransmission</type>

Commit message: debugging L_shoulder

File: Hector_ROS_Simulation/hector_description/xacro/arm.xacro (robot description, xacro)
@@ -74,4 +74,10 @@
             <dynamics damping="${damping}" friction="${friction}"/>
             <limit effort="${shoulder_torque_max}" velocity="${shoulder_velocity_max}" lower="${shoulder_min}" upper="${shoulder_max}"/>
+            <!--<xacro:if value="${(mirror_dae == True)}">
+                <limit effort="${shoulder_torque_max}" velocity="${shoulder_velocity_max}" lower="${shoulder_min}" upper="${shoulder_max}"/>
+            </xacro:if>
+            <xacro:if value="${(mirror_dae == False)}">
+                <limit effort="${shoulder_torque_max}" velocity="${shoulder_velocity_max}" lower="${shoulder_max}" upper="${shoulder_min}"/>
+            </xacro:if>  -->
         </joint>
         <link name="${name}_shoulder">

Commit message: working arms

File: Hector_ROS_Simulation/hector_description/xacro/arm.xacro (robot description, xacro)
@@ -120,7 +120,13 @@
             <parent link="${name}_shoulder"/>
             <child link="${name}_roll"/>
-            <axis xyz="0 1 0"/>
+            <axis xyz="1 0 0"/>
             <dynamics damping="${damping}" friction="${friction}"/>
             <limit effort="${shoulder_torque_max}" velocity="${shoulder_velocity_max}" lower="${shoulder_min}" upper="${shoulder_max}"/>
+            <!--<xacro:if value="${(mirror_dae == True)}">
+                <limit effort="${shoulder_torque_max}" velocity="${shoulder_velocity_max}" lower="${shoulder_min}" upper="${shoulder_max}"/>
+            </xacro:if>
+            <xacro:if value="${(mirror_dae == False)}">
+                <limit effort="${shoulder_torque_max}" velocity="${shoulder_velocity_max}" lower="${-shoulder_min}" upper="${-shoulder_max}"/>
+            </xacro:if>-->
         </joint>
         <link name="${name}_roll">

Commit message: all joints in arms work

File: Hector_ROS_Simulation/hector_description/xacro/arm.xacro (robot description, xacro)
@@ -64,8 +64,8 @@
         <joint name="${name}_shoulder_joint" type="revolute">
             <xacro:if value="${(mirror_dae == True)}">
-            <origin rpy="0 0 0" xyz="0.0 0.05 0.0"/>
+            <origin rpy="0 0 0" xyz="0.0 0.045 0.0"/>
             </xacro:if>
             <xacro:if value="${(mirror_dae == False)}">
-            <origin rpy="0 0 0" xyz="0.0 -0.05 0.0"/>
+            <origin rpy="0 0 0" xyz="0.0 -0.045 0.0"/>
             </xacro:if>
             <parent link="${name}_twist"/>
@@ -74,10 +74,4 @@
             <dynamics damping="${damping}" friction="${friction}"/>
             <limit effort="${shoulder_torque_max}" velocity="${shoulder_velocity_max}" lower="${shoulder_min}" upper="${shoulder_max}"/>
-            <!--<xacro:if value="${(mirror_dae == True)}">
-                <limit effort="${shoulder_torque_max}" velocity="${shoulder_velocity_max}" lower="${shoulder_min}" upper="${shoulder_max}"/>
-            </xacro:if>
-            <xacro:if value="${(mirror_dae == False)}">
-                <limit effort="${shoulder_torque_max}" velocity="${shoulder_velocity_max}" lower="${shoulder_max}" upper="${shoulder_min}"/>
-            </xacro:if>  -->
         </joint>
         <link name="${name}_shoulder">
@@ -113,8 +107,8 @@
         <joint name="${name}_roll_joint" type="revolute">
             <xacro:if value="${(mirror_dae == True)}">
-            <origin rpy="0 0 0" xyz="0.0 0.05 0.0"/>
+            <origin rpy="0 0 0" xyz="-0.0135 0.045 0.0"/>
             </xacro:if>
             <xacro:if value="${(mirror_dae == False)}">
-            <origin rpy="0 0 0" xyz="0.0 -0.05 0.0"/>
+            <origin rpy="0 0 0" xyz="-0.0135 -0.045 0.0"/>
             </xacro:if>
             <parent link="${name}_shoulder"/>
@@ -161,5 +155,5 @@
         </link>
         <joint name="${name}_elbow_joint" type="revolute">
-            <origin rpy="0 -1.5 0" xyz="0.0 0.0 -0.205"/>
+            <origin rpy="0 -1.5 0" xyz="${elbow_offset_x} 0.0 -0.20"/>
             <parent link="${name}_roll"/>
             <child link="${name}_elbow"/>

File: Hector_ROS_Simulation/hector_description/xacro/const.xacro (robot description, xacro)
@@ -222,5 +222,5 @@
     <xacro:property name="twist_offset_y" value="0.0"/>
     <!--xacro:property name="twist_offset_z" value="-0.22"/-->
-    <xacro:property name="twist_offset_z" value="-0.05"/>
+    <xacro:property name="twist_offset_z" value="-0.045"/>
     <xacro:property name="twist_offset" value="0.019"/>
     <xacro:property name="twist_max" value="1.4"/>
@@ -279,6 +279,6 @@
     <!-- elbow -->
     <!-- joint -->
-    <xacro:property name="elbow_offset_x" value="0.0"/>
-    <xacro:property name="elbow_offset_y" value="0.0"/>
+    <xacro:property name="elbow_offset_x" value="0.04"/>
+    <xacro:property name="elbow_offset_y" value="0.01"/>
     <xacro:property name="elbow_offset_z" value="-0.22"/>
     <xacro:property name="elbow_max" value="1.4"/>

Commit message: updated shoulder joint z offset

File: Hector_ROS_Simulation/hector_description/xacro/arm.xacro (robot description, xacro)
@@ -64,8 +64,8 @@
         <joint name="${name}_shoulder_joint" type="revolute">
             <xacro:if value="${(mirror_dae == True)}">
-            <origin rpy="0 0 0" xyz="0.0 0.045 0.0"/>
+            <origin rpy="0 0 0" xyz="0.0 0.045 -0.018"/>
             </xacro:if>
             <xacro:if value="${(mirror_dae == False)}">
-            <origin rpy="0 0 0" xyz="0.0 -0.045 0.0"/>
+            <origin rpy="0 0 0" xyz="0.0 -0.045 -0.018"/>
             </xacro:if>
             <parent link="${name}_twist"/>
